File: HexEsp-001.kicad_pcb (KiCad board)
At the start: 2 copper layers, 49.4 x 43.3 mm, 0 parts

Commit message: HexEsp Alfa Release
Parts:
- added C1: 10uF, Capacitors_SMD:C_0805, F.Cu at (213.9, 81.0)
- added C2: 10uF, Capacitors_SMD:C_0805, F.Cu at (209.7, 80.6)
- added C3: 1uF, Capacitors_SMD:C_0805, F.Cu at (209.6, 86.9)
- added C4: 10uF, Capacitors_SMD:C_0805, F.Cu at (224.9, 71.6)
- added D1: MBR120, Diodes_SMD:SOD-123, F.Cu at (222.4, 65.3)
- added D2: PURPLE, LEDs:LED_1206, F.Cu at (228.8, 65.3)
- added J1: 1x6_female_pin_Header_2.54mm, icezum:1x6-Socket-header-2.54mm, F.Cu at (178.6, 91.0)
- added J2: 1x6_female_pin_Header_2.54mm, icezum:1x6-Socket-header-2.54mm, F.Cu at (198.4, 64.9)
- added J3: 1x6_female_pin_Header_2.54mm, icezum:1x6-Socket-header-2.54mm, F.Cu at (198.4, 69.9)
- added J4: 1x6_female_pin_Header_2.54mm, icezum:1x6-Socket-header-2.54mm, F.Cu at (198.4, 75.0)
- added Q1: PZT2222A, icezum:SOT-23-3, F.Cu at (213.3, 92.1)
- added Q2: PZT2222A, icezum:SOT-23-3, F.Cu at (209.5, 91.7)
- added R1: 10K, Resistors_SMD:R_0805, F.Cu at (220.5, 77.8)
- added R2: 1K, Resistors_SMD:R_0805, F.Cu at (220.9, 71.6)
- added R3: 10K, Resistors_SMD:R_0805, F.Cu at (233.8, 65.4)
- added R4: 1K, Resistors_SMD:R_0805, F.Cu at (213.5, 87.2)
- added R5: 1K, Resistors_SMD:R_0805, F.Cu at (224.2, 77.8)
- added R6: 1K, Resistors_SMD:R_0805, F.Cu at (228.8, 71.5)
- added R7: 10K, Resistors_SMD:R_0805, F.Cu at (217.8, 84.1)
- added R8: 10K, Resistors_SMD:R_0805, F.Cu at (232.4, 71.7)
- added R9: 1K, Resistors_SMD:R_0805, F.Cu at (221.5, 84.1)
- added SW1: SW_PUSH_SMALL_H, Buttons_Switches_SMD:SW_SPST_B3U-1000P-B, F.Cu at (200.3, 91.9)
- added U1: ESP-12E, ESP8266:ESP-12E, F.Cu at (179.9, 71.3)
- added U2: SPX3819, ab2_sot:AB2_SOT23-5, F.Cu at (215.7, 74.5)
- added U3: MICRO-B_USB, Connect:USB_Micro-B, F.Cu at (202.0, 82.0)
- added U4: CP2104, Housings_DFN_QFN:QFN-24-1EP_4x4mm_Pitch0.5mm, F.Cu at (215.9, 66.7)
