File: HexEsp-001.sch (KiCad schematic (older format))
At the start: 26 parts, among them J1 1x6_female_pin_Header_2.54mm, J2 1x6_female_pin_Header_2.54mm, J3 1x6_female_pin_Header_2.54mm, J4 1x6_female_pin_Header_2.54mm, Q1 PZT2222A, Q2 PZT2222A, SW1 SW_PUSH_SMALL_H, U1 ESP-12E, U2 SPX3819, U4 MICRO-B_USB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

Commit message: HexEsp Alfa Release
Parts:
- C1, C2, C3, C4: footprint Capacitors_SMD:C_0805_HandSoldering -> Capacitors_SMD:C_0805
- D2: renamed from D3; footprint GTB2:LED_1206_Hand_Soldering -> LEDs:LED_1206
- R1, R2, R3, R4, R5, R6, R7, R8, R9: footprint Resistors_SMD:R_0805_HandSoldering -> Resistors_SMD:R_0805
- SW1: footprint Buttons_Switches_SMD:SW_SPST_TL3342 -> Buttons_Switches_SMD:SW_SPST_B3U-1000P-B
- renumbered U4 to U3, U5 to U4
Changed lines of the file:
@@
 F 0 "C1" V 1350 1775 50  0000 L CNN
 F 1 "10uF" V 1600 1725 50  0000 L CNN
-F 2 "Capacitors_SMD:C_0805_HandSoldering" H 1513 1675 50  0001 C CNN
+F 2 "Capacitors_SMD:C_0805" H 1513 1675 50  0001 C CNN
 F 3 "" H 1475 1825 50  0000 C CNN
 	1    1475 1825
@@
 F 0 "C3" V 3175 1775 50  0000 L CNN
 F 1 "1uF" V 3425 1725 50  0000 L CNN
-F 2 "Capacitors_SMD:C_0805_HandSoldering" H 3338 1675 50  0001 C CNN
+F 2 "Capacitors_SMD:C_0805" H 3338 1675 50  0001 C CNN
 F 3 "" H 3300 1825 50  0000 C CNN
 	1    3300 1825
@@
 F 0 "C2" V 2800 1775 50  0000 L CNN
 F 1 "10uF" V 3050 1750 50  0000 L CNN
-F 2 "Capacitors_SMD:C_0805_HandSoldering" H 2963 1675 50  0001 C CNN
+F 2 "Capacitors_SMD:C_0805" H 2963 1675 50  0001 C CNN
 F 3 "" H 2925 1825 50  0000 C CNN
 	1    2925 1825
@@
 F 0 "R1" V 1600 1525 50  0000 L CNN
 F 1 "10K" V 1675 1500 50  0000 L CNN
-F 2 "Resistors_SMD:R_0805_HandSoldering" V 1605 1575 50  0001 C CNN
+F 2 "Resistors_SMD:R_0805" V 1605 1575 50  0001 C CNN
 F 3 "" H 1675 1575 50  0000 C CNN
 	1    1675 1575
@@
 F 0 "R3" V 4050 1175 50  0000 L CNN
 F 1 "10K" V 4125 1150 50  0000 L CNN
-F 2 "Resistors_SMD:R_0805_HandSoldering" V 4055 1225 50  0001 C CNN
+F 2 "Resistors_SMD:R_0805" V 4055 1225 50  0001 C CNN
 F 3 "" H 4125 1225 50  0000 C CNN
 	1    4125 1225
@@
 $EndComp
 $Comp
-L MICRO-B_USB U4
+L MICRO-B_USB U3
 U 1 1 579D4052
 P 5100 1875
-F 0 "U4" H 5156 2290 50  0000 C CNN
+F 0 "U3" H 5156 2290 50  0000 C CNN
 F 1 "MICRO-B_USB" H 5156 2199 50  0000 C CNN
 F 2 "Connect:USB_Micro-B" H 5100 1875 60  0001 C CNN
@@
 F 0 "C4" V 8775 880 50  0000 L CNN
 F 1 "10uF" V 9025 830 50  0000 L CNN
-F 2 "Capacitors_SMD:C_0805_HandSoldering" H 8938 780 50  0001 C CNN
+F 2 "Capacitors_SMD:C_0805" H 8938 780 50  0001 C CNN
 F 3 "" H 8900 930 50  0000 C CNN
 	1    8900 930
@@
 F 0 "R7" V 6475 1075 50  0000 L CNN
 F 1 "10K" V 6550 1050 50  0000 L CNN
-F 2 "Resistors_SMD:R_0805_HandSoldering" V 6480 1125 50  0001 C CNN
+F 2 "Resistors_SMD:R_0805" V 6480 1125 50  0001 C CNN
 F 3 "" H 6550 1125 50  0000 C CNN
 	1    6550 1125
@@
 F 0 "R8" V 6500 1700 50  0000 L CNN
 F 1 "10K" V 6575 1675 50  0000 L CNN
-F 2 "Resistors_SMD:R_0805_HandSoldering" V 6505 1750 50  0001 C CNN
+F 2 "Resistors_SMD:R_0805" V 6505 1750 50  0001 C CNN
 F 3 "" H 6575 1750 50  0000 C CNN
 	1    6575 1750
@@
 F 0 "R4" V 5050 4400 50  0000 L CNN
 F 1 "1K" V 4975 4375 50  0000 L CNN
-F 2 "Resistors_SMD:R_0805_HandSoldering" V 4905 4450 50  0001 C CNN
+F 2 "Resistors_SMD:R_0805" V 4905 4450 50  0001 C CNN
 F 3 "" H 4975 4450 50  0000 C CNN
 	1    4975 4450
@@
 F 0 "R5" V 5350 4400 50  0000 L CNN
 F 1 "1K" V 5275 4375 50  0000 L CNN
-F 2 "Resistors_SMD:R_0805_HandSoldering" V 5205 4450 50  0001 C CNN
+F 2 "Resistors_SMD:R_0805" V 5205 4450 50  0001 C CNN
 F 3 "" H 5275 4450 50  0000 C CNN
 	1    5275 4450
@@
 F 0 "R6" V 5650 4400 50  0000 L CNN
 F 1 "1K" V 5575 4375 50  0000 L CNN
-F 2 "Resistors_SMD:R_0805_HandSoldering" V 5505 4450 50  0001 C CNN
+F 2 "Resistors_SMD:R_0805" V 5505 4450 50  0001 C CNN
 F 3 "" H 5575 4450 50  0000 C CNN
 	1    5575 4450
@@
 F 0 "R9" V 9450 4475 50  0000 L CNN
 F 1 "1K" V 9375 4450 50  0000 L CNN
-F 2 "Resistors_SMD:R_0805_HandSoldering" V 9305 4525 50  0001 C CNN
+F 2 "Resistors_SMD:R_0805" V 9305 4525 50  0001 C CNN
 F 3 "" H 9375 4525 50  0000 C CNN
 	1    9375 4525
@@
 GPIO0
 $Comp
-L LED D3
+L LED D2
 U 1 1 579E74FA
 P 9375 4075
-F 0 "D3" H 9425 4200 50  0000 R CNN
+F 0 "D2" H 9425 4200 50  0000 R CNN
 F 1 "PURPLE" H 9500 3950 50  0000 R CNN
-F 2 "GTB2:LED_1206_Hand_Soldering" H 9375 4075 50  0001 C CNN
+F 2 "LEDs:LED_1206" H 9375 4075 50  0001 C CNN
 F 3 "" H 9375 4075 50  0000 C CNN
 	1    9375 4075
@@
 GND
 $Comp
-L CP2104 U5
+L CP2104 U4
 U 1 1 57F3E58E
 P 9930 1690
-F 0 "U5" H 9930 1870 60  0000 C CNN
+F 0 "U4" H 9930 1870 60  0000 C CNN
 F 1 "CP2104" H 9920 1750 60  0000 C CNN
 F 2 "Housings_DFN_QFN:QFN-24-1EP_4x4mm_Pitch0.5mm" H 9930 1490 60  0001 C CNN
@@
 F 0 "R2" V 3875 4300 50  0000 L CNN
 F 1 "1K" V 3800 4275 50  0000 L CNN
-F 2 "Resistors_SMD:R_0805_HandSoldering" V 3730 4350 50  0001 C CNN
+F 2 "Resistors_SMD:R_0805" V 3730 4350 50  0001 C CNN
 F 3 "" H 3800 4350 50  0000 C CNN
 	1    3800 4350
@@
 F 0 "SW1" V 4171 1735 50  0000 R CNN
 F 1 "SW_PUSH_SMALL_H" V 4080 1735 50  0000 R CNN
-F 2 "Buttons_Switches_SMD:SW_SPST_TL3342" H 4125 1975 50  0001 C CNN
+F 2 "Buttons_Switches_SMD:SW_SPST_B3U-1000P-B" H 4125 1975 50  0001 C CNN
 F 3 "" H 4125 1975 50  0000 C CNN
 	1    4125 1775
