File: ch340/HexEsp-001.sch (KiCad schematic (older format))
At the start: 28 parts, among them IC1 CH340G, J1 1x6_female_pin_Header_2.54mm, J2 1x6_female_pin_Header_2.54mm, J3 1x6_female_pin_Header_2.54mm, J4 1x6_female_pin_Header_2.54mm, Q1 PZT2222A, Q2 PZT2222A, U1 ESP-12E, U2 SPX3819, U3 PUSHBUTTON, U4 MICRO-B_USB

Commit message: Re-organized directory
Parts:
- removed D1: MBR120, Diodes_SMD:SOD-123, symbol D_Schottky
- removed U3: PUSHBUTTON, makerlab:PUSHBUTTON_SMD_PTS810, symbol PUSHBUTTON
- added C4: 10uF, Capacitors_SMD:C_0805, symbol C
- added C6: 100nF, Capacitors_SMD:C_0805, symbol C
- added D1: MBR120, Diodes_SMD:SOD-123, symbol D_Schottky_Small
- added SW1: RESET, Buttons_Switches_SMD:SW_SPST_B3U-1000P-B, symbol SW_PUSH_SMALL_H
- C1: footprint Capacitors_SMD:C_0805_HandSoldering -> Capacitors_SMD:C_0805
- C2: value 1uF -> 10uF; footprint Capacitors_SMD:C_0805_HandSoldering -> Capacitors_SMD:C_0805
- C3: value 10uF -> 1uF; footprint Capacitors_SMD:C_0805_HandSoldering -> Capacitors_SMD:C_0805
- C5: renamed from C4; value 10uF -> 100nF; footprint Capacitors_SMD:C_0805_HandSoldering -> Capacitors_SMD:C_0805
- D2: renamed from D3; footprint GTB2:LED_1206_Hand_Soldering -> LEDs:LED_1206
- IC1: footprint Housings_SOIC:SOIC-16_3.9x9.9mm_Pitch1.27mm -> CH340G:SOP-16; symbol CH340G -> CH340G-RESCUE-HexEsp-001
- Q1, Q2: footprint MazEsp-001:AB2_SOT23-3 -> ab2_sot:AB2_SOT23-3
- R1, R4: footprint Resistors_SMD:R_0805_HandSoldering -> Resistors_SMD:R_0805
- R10: renamed from R13; footprint Resistors_SMD:R_0805_HandSoldering -> Resistors_SMD:R_0805
- R2: renamed from R3; footprint Resistors_SMD:R_0805_HandSoldering -> Resistors_SMD:R_0805
- R3: renamed from R7; footprint Resistors_SMD:R_0805_HandSoldering -> Resistors_SMD:R_0805
- R5: renamed from R8; footprint Resistors_SMD:R_0805_HandSoldering -> Resistors_SMD:R_0805
- R6: renamed from R5; footprint Resistors_SMD:R_0805_HandSoldering -> Resistors_SMD:R_0805
- R7: renamed from R6; footprint Resistors_SMD:R_0805_HandSoldering -> Resistors_SMD:R_0805
- R8: renamed from R9; footprint Resistors_SMD:R_0805_HandSoldering -> Resistors_SMD:R_0805
- R9: renamed from R12; footprint Resistors_SMD:R_0805_HandSoldering -> Resistors_SMD:R_0805
- RES1: footprint makerlab:RESONATOR_CSTCE -> Resonators:murata-resonator_SMD_CSTCE8M00G55-R0
- renumbered U4 to U3
Connections:
- net labels removed: 3V3, VIN
- wire segments 116 -> 112
- no-connect marks 14 -> 15
Other:
- note added: "RESET & AUTORESET"
- note removed: "RESET"
- moved on the sheet: C1, Q1, Q2, R3, R5, RES1, U3

Commit message: Some litle changes
Parts:
- renumbered D2 to D1, D1 to D2, R8 to R3, R3 to R4, R4 to R6, R6 to R7, R7 to R8
Connections:
- wire segments 112 -> 110
- no-connect marks 15 -> 17
Other:
- note added: "ESP8266 CORE"
- note added: "LED"
- note added: "PINOUT"
- moved on the sheet: D1, J1, J2, J3, J4, Q1, Q2, R2, R3, R4, R5, R6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
